File: RaspberryPiBreakout_Hardware/RaspberryPiBreakout_Hardware/RaspberryPiBreakout_Hardware.kicad_pcb (KiCad board)
At the start: 2 copper layers, 5 parts, among them U1 OKI, U2 Raspberry_Pi

Commit message: finished Layout
Parts:
- added G***: LOGO, MRDT_Silkscreens:2_Dahlbot_2.0, B.Cu at (145.3, 99.1)
- added G***: LOGO, MRDT_Silkscreens:0_MRDT_Logo_30mm, F.Cu at (99.6, 98.6)
- added G***: LOGO, MRDT_Silkscreens:z_sig_Andrew_Van_Horn_Sig_15mm, F.Cu at (86.4, 144.8)
- moved U2 102.1 mm to (72.4, 128.3)
- moved C2 87.2 mm to (157.5, 116.4), turned to 90 degrees
- moved C1 73.1 mm to (157.5, 112.2), turned to 270 degrees
- moved U1 58.7 mm to (153.7, 109.2), turned to 270 degrees
- moved Conn1 57.4 mm to (171.2, 106.7), turned to 180 degrees
Routing:
- net +5V: track 0.00 -> 80.4 mm
- net Net-(C1-Pad1): track 0.00 -> 15.7 mm
- added copper zone on B.Cu, net GND
- added copper zone on F.Cu, net GND
Other:
- board outline added: 124.5 x 79.2 mm
- board text added: "5V"
- board text added: "Raspberry Pi Breakout, Rev 1 Mars Rover Design Team Missouri S&T, 2019 Andrew Van Horn"
